File: Block Relay.kicad_sch (KiCad schematic)
At the start: 25 parts, among them J14 Screw_Terminal_01x02, J15 Screw_Terminal_01x02, J16 Screw_Terminal_01x02, J17 Screw_Terminal_01x02, J18 Screw_Terminal_01x02, K10 SRD-05VDC-SL-C, K5 SRD-05VDC-SL-C, K7 SRD-05VDC-SL-C, K8 SRD-05VDC-SL-C, K9 SRD-05VDC-SL-C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

Commit message: refactored project and fix some bugs
Other:
- moved on the sheet: J15, J16, J17, J18, K10, K7, K8, K9, R9
