File: HydroB.kicad_sch (KiCad schematic)
At the start: 0 parts

Commit message: refactored project and fix some bugs
Other:
- sheet ESP32-S4 renamed ESP32-S3
- sheet Power Supply1 renamed Power Supply
- sheet Block Relay1 ports: added none; removed 5V, GND
- sheet ESP32-S3 ports: added none; removed 3.3V, GND
- sheet Power Supply ports: added none; removed 3.3V, 5V, GND, VBUS
