File: HydroB V2_SubBoard/Block Relay.kicad_sch (KiCad schematic)
At the start: 25 parts, among them J14 Screw_Terminal_01x02, J15 Screw_Terminal_01x02, J16 Screw_Terminal_01x02, J17 Screw_Terminal_01x02, J18 Screw_Terminal_01x02, K10 SRD-05VDC-SL-C, K5 SRD-05VDC-SL-C, K7 SRD-05VDC-SL-C, K8 SRD-05VDC-SL-C, K9 SRD-05VDC-SL-C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

Commit message: the schematic of sub-board updated
Parts:
- K10, K5, K7, K8, K9: footprint SRD-05VDC-SL-C:RELAY_SRD-05VDC-SL-C -> SRD-05VDC-SL-C (1):RELAY_SRD-05VDC-SL-C
Changed lines of the file:
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@@
 			)
 		)
-		(property "Footprint" "SRD-05VDC-SL-C:RELAY_SRD-05VDC-SL-C"
+		(property "Footprint" "SRD-05VDC-SL-C (1):RELAY_SRD-05VDC-SL-C"
 			(at 192.278 114.3 0)
 			(effects
@@
 			)
 		)
-		(property "Footprint" "SRD-05VDC-SL-C:RELAY_SRD-05VDC-SL-C"
+		(property "Footprint" "SRD-05VDC-SL-C (1):RELAY_SRD-05VDC-SL-C"
 			(at 212.598 60.96 0)
 			(effects
@@
 			)
 		)
-		(property "Footprint" "SRD-05VDC-SL-C:RELAY_SRD-05VDC-SL-C"
+		(property "Footprint" "SRD-05VDC-SL-C (1):RELAY_SRD-05VDC-SL-C"
 			(at 104.648 114.3 0)
 			(effects
@@
 			)
 		)
-		(property "Footprint" "SRD-05VDC-SL-C:RELAY_SRD-05VDC-SL-C"
+		(property "Footprint" "SRD-05VDC-SL-C (1):RELAY_SRD-05VDC-SL-C"
 			(at 146.558 60.96 0)
 			(effects
@@
 			)
 		)
-		(property "Footprint" "SRD-05VDC-SL-C:RELAY_SRD-05VDC-SL-C"
+		(property "Footprint" "SRD-05VDC-SL-C (1):RELAY_SRD-05VDC-SL-C"
 			(at 77.47 60.96 0)
 			(effects
