File: HydroB V2_Mainboard/High speed.kicad_sch (KiCad schematic)
At the start: 12 parts, among them U5 74VHC86M

Commit message: Mainboard schematic update
Parts:
- added R6: 510R, Resistor_SMD:R_0603_1608Metric, symbol Device:R
- D1, D5: footprint Package_TO_SOT_SMD:SOT-353_SC-70-5 -> Diode_SMD:D_SOD-123F
- R24: value 510R -> 220k
Connections:
- net BUSY: now also R6.1; no longer U5.3 (O0)
- new net: R6.2, U5.3 (O0)
- no-connect marks 1 -> 3
Other:
- moved on the sheet: C17, D5A, R18
Changed lines of the file:
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@@
 	)
 	(junction
-		(at 177.8 95.25)
+		(at 175.26 81.28)
 		(diameter 0)
 		(color 0 0 0 0)
@@
 	)
 	(junction
-		(at 167.64 81.28)
+		(at 185.42 95.25)
 		(diameter 0)
 		(color 0 0 0 0)
@@
 	)
 	(no_connect
+		(at 121.92 88.9)
+	)
+	(no_connect
+		(at 121.92 93.98)
+	)
+	(no_connect
 		(at 157.48 86.36)
 	)
@@
 	(wire
 		(pts
-			(xy 186.69 81.28) (xy 181.61 81.28)
+			(xy 195.58 81.28) (xy 189.23 81.28)
 		)
 		(stroke
@@
 	(wire
 		(pts
-			(xy 186.69 95.25) (xy 177.8 95.25)
+			(xy 195.58 95.25) (xy 185.42 95.25)
 		)
 		(stroke
@@
 	(wire
 		(pts
+			(xy 158.75 83.82) (xy 157.48 83.82)
+		)
+		(stroke
+			(width 0)
+			(type default)
+		)
+	)
+	(wire
+		(pts
+			(xy 167.64 83.82) (xy 166.37 83.82)
+		)
+		(stroke
+			(width 0)
+			(type default)
+		)
+	)
+	(wire
+		(pts
 			(xy 109.22 104.14) (xy 111.76 104.14)
 		)
@@
 	(wire
 		(pts
-			(xy 167.64 95.25) (xy 177.8 95.25)
+			(xy 175.26 95.25) (xy 185.42 95.25)
 		)
 		(stroke
@@
 	(wire
 		(pts
-			(xy 186.69 92.71) (xy 186.69 95.25)
-		)
-		(stroke
-			(width 0)
-			(type default)
-		)
-	)
-	(wire
-		(pts
-			(xy 157.48 81.28) (xy 167.64 81.28)
+			(xy 195.58 92.71) (xy 195.58 95.25)
+		)
+		(stroke
+			(width 0)
+			(type default)
+		)
+	)
+	(wire
+		(pts
+			(xy 157.48 81.28) (xy 175.26 81.28)
 		)
 		(stroke
@@
 	(wire
 		(pts
-			(xy 167.64 81.28) (xy 167.64 86.36)
+			(xy 175.26 81.28) (xy 175.26 86.36)
 		)
 		(stroke
@@
 	(wire
 		(pts
-			(xy 167.64 91.44) (xy 167.64 95.25)
+			(xy 175.26 91.44) (xy 175.26 95.25)
+		)
+		(stroke
+			(width 0)
+			(type default)
+		)
+	)
+	(wire
+		(pts
+			(xy 175.26 81.28) (xy 181.61 81.28)
 		)
 		(stroke
@@
 	(wire
 		(pts
-			(xy 111.76 127) (xy 111.76 125.73)
+			(xy 111.76 127) (xy 111.76 129.54)
 		)
 		(stroke
@@
 	(wire
 		(pts
-			(xy 186.69 85.09) (xy 186.69 81.28)
+			(xy 195.58 85.09) (xy 195.58 81.28)
 		)
 		(stroke
@@
 		(pts
 			(xy 104.14 90.17) (xy 104.14 92.71)
-		)
-		(stroke
-			(width 0)
-			(type default)
-		)
-	)
-	(wire
-		(pts
-			(xy 167.64 81.28) (xy 173.99 81.28)
 		)
 		(stroke
@@
 	(text "High Speed operation\n"
 		(exclude_from_sim no)
-		(at 169.672 126.492 0)
+		(at 168.148 124.206 0)
 		(effects
 			(font
@@
 	(hierarchical_label "BUSY"
 		(shape input)
-		(at 157.48 83.82 0)
+		(at 167.64 83.82 0)
 		(fields_autoplaced yes)
 		(effects
@@
 	(symbol
 		(lib_id "power:GND")
-		(at 177.8 95.25 0)
+		(at 185.42 95.25 0)
 		(unit 1)
 		(exclude_from_sim no)
@@
 		(fields_autoplaced yes)
 		(property "Reference" "#PWR01"
-			(at 177.8 101.6 0)
+			(at 185.42 101.6 0)
 			(effects
 				(font
@@
 		)
 		(property "Value" "GND"
-			(at 177.8 100.33 0)
+			(at 185.42 100.33 0)
 			(effects
 				(font
@@
 		)
 		(property "Footprint" ""
-			(at 177.8 95.25 0)
+			(at 185.42 95.25 0)
 			(effects
 				(font
@@
 		)
 		(property "Datasheet" ""
-			(at 177.8 95.25 0)
+			(at 185.42 95.25 0)
 			(effects
 				(font
@@
 		)
 		(property "Description" "Power symbol creates a global label with name \"GND\" , ground"
-			(at 177.8 95.25 0)
+			(at 185.42 95.25 0)
 			(effects
 				(font
@@
 				(path "/7eaed49e-949c-4b32-bb59-42041e199453/cb3a589e-3872-4cde-9770-3d39d4934022/745861c9-38a8-465b-931f-39bedf809fd4"
 					(reference "#PWR01")
+					(unit 1)
+				)
+			)
+		)
+	)
+	(symbol
+		(lib_id "Device:R")
+		(at 162.56 83.82 270)
+		(unit 1)
+		(exclude_from_sim no)
+		(in_bom yes)
+		(on_board yes)
+		(dnp no)
+		(property "Reference" "R6"
+			(at 162.56 86.106 90)
+			(effects
+				(font
+					(size 1.27 1.27)
+				)
+			)
+		)
+		(property "Value" "510R"
+			(at 162.56 88.138 90)
+			(effects
+				(font
+					(size 1.27 1.27)
+				)
+			)
+		)
+		(property "Footprint" "Resistor_SMD:R_0603_1608Metric"
+			(at 162.56 82.042 90)
+			(effects
+				(font
+					(size 1.27 1.27)
+				)
+				(hide yes)
+			)
+		)
+		(property "Datasheet" "~"
+			(at 162.56 83.82 0)
+			(effects
+				(font
+					(size 1.27 1.27)
+				)
+				(hide yes)
+			)
+		)
+		(property "Description" "Resistor"
+			(at 162.56 83.82 0)
+			(effects
+				(font
+					(size 1.27 1.27)
+				)
+				(hide yes)
+			)
+		)
+		(pin "2"
+		)
+		(pin "1"
+		)
+		(instances
+			(project "LCD High Revolution"
+				(path "/7eaed49e-949c-4b32-bb59-42041e199453/cb3a589e-3872-4cde-9770-3d39d4934022/745861c9-38a8-465b-931f-39bedf809fd4"
+					(reference "R6")
 					(unit 1)
 				)
@@
 			)
 		)
-		(property "Value" "510R"
+		(property "Value" "220k"
 			(at 105.41 108.712 90)
 			(effects
@@
 	(symbol
 		(lib_id "Device:C")
-		(at 186.69 88.9 0)
+		(at 195.58 88.9 0)
 		(unit 1)
 		(exclude_from_sim no)
@@
 		(fields_autoplaced yes)
 		(property "Reference" "C17"
-			(at 190.5 87.6299 0)
+			(at 199.39 87.6299 0)
 			(effects
 				(font
@@
 		)
 		(property "Value" "1nF"
-			(at 190.5 90.1699 0)
+			(at 199.39 90.1699 0)
 			(effects
 				(font
@@
 		)
 		(property "Footprint" "Capacitor_SMD:C_0603_1608Metric"
-			(at 187.6552 92.71 0)
+			(at 196.5452 92.71 0)
 			(effects
 				(font
@@
 		)
 		(property "Datasheet" "~"
-			(at 186.69 88.9 0)
+			(at 195.58 88.9 0)
 			(effects
 				(font
@@
 		)
 		(property "Description" "Unpolarized capacitor"
-			(at 186.69 88.9 0)
+			(at 195.58 88.9 0)
 			(effects
 				(font
@@
 	(symbol
 		(lib_id "Power_Protection:PESD3V3L4UG")
-		(at 167.64 88.9 90)
+		(at 175.26 88.9 90)
 		(unit 1)
 		(exclude_from_sim no)
@@
 		(fields_autoplaced yes)
 		(property "Reference" "D5"
-			(at 170.18 87.6299 90)
+			(at 177.8 87.6299 90)
 			(effects
 				(font
@@
 		)
 		(property "Value" "PESD3V3L4UG"
-			(at 170.18 90.1699 90)
+			(at 177.8 90.1699 90)
 			(effects
 				(font
@@
 			)
 		)
-		(property "Footprint" "Package_TO_SOT_SMD:SOT-353_SC-70-5"
-			(at 162.56 88.9 0)
+		(property "Footprint" "Diode_SMD:D_SOD-123F"
+			(at 170.18 88.9 0)
 			(effects
 				(font
@@
 		)
 		(property "Datasheet" "https://assets.nexperia.com/documents/data-sheet/PESDXL4UF_G_W.pdf"
-			(at 172.72 88.9 0)
+			(at 180.34 88.9 0)
 			(effects
 				(font
@@
 		)
 		(property "Description" "Low capacitance unidirectional quadruple ESD protection diode array, 3.3V, Common Anode, SOT-353"
-			(at 167.64 88.9 0)
+			(at 175.26 88.9 0)
 			(effects
 				(font
@@
 			)
 		)
-		(property "Footprint" "Package_TO_SOT_SMD:SOT-353_SC-70-5"
+		(property "Footprint" "Diode_SMD:D_SOD-123F"
 			(at 102.87 111.76 0)
 			(effects
@@
 		(dnp no)
 		(property "Reference" "R1"
-			(at 104.902 94.488 90)
+			(at 104.902 94.234 90)
 			(effects
 				(font
@@
 	(symbol
 		(lib_id "power:GND")
-		(at 111.76 125.73 0)
+		(at 111.76 129.54 0)
 		(unit 1)
 		(exclude_from_sim no)
@@
 		(dnp no)
 		(property "Reference" "#PWR040"
-			(at 111.76 132.08 0)
+			(at 111.76 135.89 0)
 			(effects
 				(font
@@
 		)
 		(property "Value" "GND"
-			(at 114.046 130.048 0)
+			(at 114.046 133.858 0)
 			(effects
 				(font
@@
 		)
 		(property "Footprint" ""
-			(at 111.76 125.73 0)
+			(at 111.76 129.54 0)
 			(effects
 				(font
@@
 		)
 		(property "Datasheet" ""
-			(at 111.76 125.73 0)
+			(at 111.76 129.54 0)
 			(effects
 				(font
@@
 		)
 		(property "Description" "Power symbol creates a global label with name \"GND\" , ground"
-			(at 111.76 125.73 0)
+			(at 111.76 129.54 0)
 			(effects
 				(font
@@
 	(symbol
 		(lib_id "Device:R")
-		(at 177.8 81.28 270)
+		(at 185.42 81.28 270)
 		(unit 1)
 		(exclude_from_sim no)
@@
 		(dnp no)
 		(property "Reference" "R18"
-			(at 177.8 83.566 90)
+			(at 185.42 83.566 90)
 			(effects
 				(font
@@
 		)
 		(property "Value" "220R"
-			(at 177.8 85.598 90)
+			(at 185.42 85.598 90)
 			(effects
 				(font
@@
 		)
 		(property "Footprint" "Resistor_SMD:R_0603_1608Metric"
-			(at 177.8 79.502 90)
+			(at 185.42 79.502 90)
 			(effects
 				(font
@@
 		)
 		(property "Datasheet" "~"
-			(at 177.8 81.28 0)
+			(at 185.42 81.28 0)
 			(effects
 				(font
@@
 		)
 		(property "Description" "Resistor"
-			(at 177.8 81.28 0)
-			(effects
-				(font
+			(at 185.42 81.28 0)
+			(effects
+				(font
