File: HydroB V2_Mainboard/LCD High Revolution.kicad_pcb (KiCad board)
At the start: 2 copper layers, 76.5 x 71.3 mm, 70 parts, among them J1 Conn_01x42_Pin, J2 Conn_01x08_Pin, J3 Conn_01x02_Pin, J4 Conn_01x02_Pin, J5 USB_C_Receptacle_USB2.0_16P, Q1 S8050, SW1 SW_Push, SW2 SW_Push, U1 ESP32-S3-WROOM-1-N16R2, U3 TPS562200, U4 SN65HVD230

Commit message: Mainboard schematic update
Parts:
- removed C1, C3, C32, C34, C43, C45: 0.1uF, Capacitor_SMD:C_0603_1608Metric
- removed C2, C27, C31, C33, C41, C42: 10uF, Capacitor_SMD:C_0603_1608Metric
- removed C28: 10pF/50V, Capacitor_SMD:C_0805_2012Metric
- removed C29: 4.7uF/35V, Capacitor_Tantalum_SMD:CP_EIA-7343-43_Kemet-X_Pad2.25x2.55mm_HandSolder
- removed C30: 0.1uF/50V, Capacitor_Tantalum_SMD:CP_EIA-7343-43_Kemet-X_Pad2.25x2.55mm_HandSolder
- removed C37: NC, Capacitor_SMD:C_0603_1608Metric
- removed C38: 18pF, Capacitor_SMD:C_0603_1608Metric
- removed C39, C44: 22uF, Capacitor_SMD:C_0603_1608Metric
- removed C4: 0.1uF/10V, Capacitor_SMD:C_0805_2012Metric
- removed C40: 100nF, Capacitor_SMD:C_0603_1608Metric
- removed C46: 4.7uF/6.3V, Capacitor_SMD:C_0805_2012Metric
- removed C47: 22pF/50V, Capacitor_SMD:C_0805_2012Metric
- removed D1, D8: LED_Small, LED_SMD:LED_0805_2012Metric
- removed D7: 1N4148WS, Diode_SMD:D_SOD-323
- removed H1, H2, H3, H4: MountingHole, MountingHole:MountingHole_3mm_Pad_Via
- removed J1: Conn_01x42_Pin, Connector_FFC-FPC:Hirose_FH12-40S-0.5SH_1x40-1MP_P0.50mm_Horizontal
- removed J2: Conn_01x08_Pin, Connector_FFC-FPC:Hirose_FH12-6S-0.5SH_1x06-1MP_P0.50mm_Horizontal
- removed J3, J4: Conn_01x02_Pin, Connector_JST:JST_XH_B2B-XH-A_1x02_P2.50mm_Vertical
- removed J5: USB_C_Receptacle_USB2.0_16P, Connector_USB:USB_C_Receptacle_G-Switch_GT-USB-7010ASV
- removed L3: 10uH, Inductor_SMD:L_Bourns_SRP5030T
- removed L4: 4.7uH, Inductor_SMD:L_Bourns_SRP5030T
- removed Q1: S8050, Package_TO_SOT_THT:TO-92_Inline
- removed R1, R32: 1k, Resistor_SMD:R_0603_1608Metric
- removed R18, R23: NC, Resistor_SMD:R_0603_1608Metric
- removed R19, R20: 10K, Resistor_SMD:R_0603_1608Metric
- removed R2, R3, R30, R31, R6: 10k, Resistor_SMD:R_0603_1608Metric
- removed R21: 50R, Resistor_SMD:R_0603_1608Metric
- removed R22: 3.6R, Resistor_SMD:R_0603_1608Metric
- removed R24, R26, R27, R4: NC, Resistor_SMD:R_0402_1005Metric
- removed R25: 10k, Resistor_SMD:R_0402_1005Metric
- removed R28, R29: 5.1K, Resistor_SMD:R_0402_1005Metric
- removed R33: 100k, Resistor_SMD:R_0603_1608Metric
- removed R34: 30k, Resistor_SMD:R_0603_1608Metric
- removed R35: R, Resistor_SMD:R_0603_1608Metric
- removed R36: 120, Resistor_SMD:R_0603_1608Metric
- removed R37: 135k, Resistor_SMD:R_0603_1608Metric
- removed R5: 0R, Resistor_SMD:R_0402_1005Metric
- removed RY1: ~, Package_TO_SOT_SMD:SOT-23-6
- removed SW1, SW2: SW_Push, Button_Switch_SMD:SW_Push_SPST_NO_Alps_SKRK
- removed U1: ESP32-S3-WROOM-1-N16R2, MOD FILE:XCVR_ESP32-S3-WROOM-1-N16R2
- removed U3: TPS562200, Package_TO_SOT_SMD:SOT-23-6
- removed U4: SN65HVD230, Package_SO:SOIC-8_3.9x4.9mm_P1.27mm
Other:
- board outline removed

Commit message: main PCB board placement
Parts:
- added C1: 0.1uF, Capacitor_SMD:C_0603_1608Metric, F.Cu at (156.7, 65.5)
- added C10: 22uF, Capacitor_SMD:C_0805_2012Metric, F.Cu at (114.9, 83.2)
- added C11: 22uF, Capacitor_SMD:C_0805_2012Metric, F.Cu at (117.5, 83.2)
- added C12: 22uF, Capacitor_SMD:C_0805_2012Metric, F.Cu at (120.0, 83.2)
- added C13: 22uF, Capacitor_SMD:C_0805_2012Metric, F.Cu at (122.5, 83.2)
- added C14: 1uF, Capacitor_SMD:C_0805_2012Metric, F.Cu at (141.7, 77.1)
- added C15: 1uF, Capacitor_SMD:C_0805_2012Metric, F.Cu at (139.0, 82.8)
- added C16: 1uF, Capacitor_SMD:C_0603_1608Metric, F.Cu at (135.8, 110.8)
- added C17: 100nF, Capacitor_SMD:C_0603_1608Metric, F.Cu at (135.8, 112.7)
- added C18: 100nF, Capacitor_SMD:C_0603_1608Metric, F.Cu at (135.5, 109.0)
- added C2: 10uF, Capacitor_SMD:C_0603_1608Metric, F.Cu at (155.9, 62.1)
- added C3: 100nF, Capacitor_SMD:C_0603_1608Metric, F.Cu at (157.9, 62.1)
- added C4: 10uF, Capacitor_SMD:CP_Elec_4x3, F.Cu at (94.8, 92.3)
- added C5: 0.1uF, Capacitor_SMD:C_0603_1608Metric, F.Cu at (115.8, 117.9)
- added C6: 220nF, Capacitor_SMD:C_0805_2012Metric, F.Cu at (100.9, 91.1)
- added C7: 1uF, Capacitor_SMD:C_0805_2012Metric, F.Cu at (116.5, 93.3)
- added C8: 100NF, Capacitor_SMD:C_0603_1608Metric, F.Cu at (115.6, 90.5)
- added C9: c, Capacitor_SMD:C_0805_2012Metric, F.Cu at (115.6, 100.8)
- added D1: LED_Small, LED_SMD:LED_0805_2012Metric, F.Cu at (186.3, 64.6)
- added D3: LEDR, LED_SMD:LED_0603_1608Metric, F.Cu at (150.1, 105.5)
- added D4: D_TVS, Diode_SMD:D_SOD-123F, F.Cu at (107.1, 113.0)
- added D5: LEDR, LED_SMD:LED_0603_1608Metric, F.Cu at (150.1, 111.1)
- added D8: LED_Small, LED_SMD:LED_0805_2012Metric, F.Cu at (135.0, 75.9)
- added F1: Fuse, Fuse:Fuse_0805_2012Metric, F.Cu at (139.7, 118.4)
- added G***: LOGO, CHIPTREE_LOGO:CHPTREE-10x10mm, F.Cu at (165.8, 99.8)
- added G***: LOGO, CHIPTREE_LOGO:cam10x10, F.Cu at (177.4, 98.7)
- added J1: Conn_01x02_Pin, DC Conn:Modbus, F.Cu at (83.6, 97.1)
- added J10: USB_C_2.0, Connector_USB:USB_C_Receptacle_Palconn_UTC16-G, F.Cu at (138.9, 60.4)
- added J2: Conn_01x02_Pin, Connector_JST:JST_EH_B2B-EH-A_1x02_P2.50mm_Vertical, F.Cu at (97.9, 60.5)
- added J3: SENSOR, DC Conn:Modbus, F.Cu at (104.0, 127.4)
- added J4: Conn_01x02_Pin, Connector_JST:JST_EH_B2B-EH-A_1x02_P2.50mm_Vertical, F.Cu at (110.8, 60.5)
- added J6: 12V, DC Conn:DC conn, F.Cu at (79.1, 78.1)
- added J7: Conn_01x02_Pin, Connector_PinHeader_2.00mm:PinHeader_1x02_P2.00mm_Vertical, F.Cu at (125.7, 84.2)
- added J8: LCD, Connector_JST:JST_EH_B2B-EH-A_1x02_P2.50mm_Vertical, F.Cu at (123.0, 60.5)
- added J9: SENSOR, DC Conn:Modbus, F.Cu at (179.1, 127.4)
- added L1: 10uH, Inductor_SMD:L_Bourns_SRP5030T, F.Cu at (107.2, 83.9)
- added Q1: S8050, Package_TO_SOT_SMD:SOT-23, F.Cu at (94.8, 70.1)
- added Q2: S8050, Package_TO_SOT_SMD:SOT-23, F.Cu at (107.8, 70.2)
- added Q3: 1P, Package_TO_SOT_SMD:SOT-23, F.Cu at (143.1, 99.1)
- added Q4: 1P, Package_TO_SOT_SMD:SOT-23, F.Cu at (136.1, 99.1)
- added R1: 1k, Resistor_SMD:R_0603_1608Metric, F.Cu at (184.1, 64.6)
- added R10: 2.1k, Resistor_SMD:R_0603_1608Metric, F.Cu at (112.0, 110.0)
- added R11: 120, Resistor_SMD:R_0603_1608Metric, F.Cu at (103.2, 113.0)
- added R12: 100k, Resistor_SMD:R_0603_1608Metric, F.Cu at (113.0, 100.8)
- added R13: 43.2k, Resistor_SMD:R_0603_1608Metric, F.Cu at (111.9, 97.5)
- added R14: 10K, Resistor_SMD:R_0603_1608Metric, F.Cu at (142.7, 87.3)
- added R15: 1.96M, Resistor_SMD:R_0402_1005Metric, F.Cu at (142.2, 85.0)
- added R16: 1.18M, Resistor_SMD:R_0402_1005Metric, F.Cu at (144.4, 85.0)
- added R18: 10k, Resistor_SMD:R_0603_1608Metric, F.Cu at (142.1, 116.9)
- added R19: 10k, Resistor_SMD:R_0603_1608Metric, F.Cu at (139.0, 99.5)
- added R20: 10k, Resistor_SMD:R_0603_1608Metric, F.Cu at (145.9, 99.5)
- added R21: 1k, Resistor_SMD:R_0603_1608Metric, F.Cu at (150.1, 107.3)
- added R22: 1k, Resistor_SMD:R_0603_1608Metric, F.Cu at (150.1, 109.3)
- added R3: Variable Resistor, Resistor_SMD:R_0603_1608Metric, F.Cu at (98.7, 69.1)
- added R30: 10k, Resistor_SMD:R_0603_1608Metric, F.Cu at (156.7, 67.8)
- added R31: 10k, Resistor_SMD:R_0603_1608Metric, F.Cu at (183.2, 78.2)
- added R32: 1k, Resistor_SMD:R_0603_1608Metric, F.Cu at (135.0, 78.3)
- added R4: 10K, Resistor_SMD:R_0603_1608Metric, F.Cu at (98.8, 71.1)
- added R5: 100k, Resistor_SMD:R_0603_1608Metric, F.Cu at (105.8, 97.4)
- added R6: Variable Resistor, Resistor_SMD:R_0603_1608Metric, F.Cu at (111.7, 69.2)
- added R7: 10K, Resistor_SMD:R_0603_1608Metric, F.Cu at (111.7, 71.2)
- added R8: 2.1k, Resistor_SMD:R_0603_1608Metric, F.Cu at (112.0, 116.0)
- added R9: 124, Resistor_SMD:R_0603_1608Metric, F.Cu at (111.2, 113.0)
- added SW1: SW_Push, Button_Switch_THT:SW_Tactile_SPST_Angled_PTS645Vx39-2LFS, F.Cu at (75.0, 120.7)
- added SW2: SW_Push, Button_Switch_SMD:SW_Push_SPST_NO_Alps_SKRK, F.Cu at (187.2, 71.6)
- added TP1: TestPoint, TestPoint:TestPoint_Loop_D1.80mm_Drill1.0mm_Beaded, F.Cu at (97.3, 115.5)
- added TP2: TestPoint, TestPoint:TestPoint_Loop_D1.80mm_Drill1.0mm_Beaded, F.Cu at (97.3, 110.8)
- added TP3: TestPoint, TestPoint:TestPoint_Loop_D1.80mm_Drill1.0mm_Beaded, F.Cu at (153.1, 72.0)
- added TP4: TestPoint, TestPoint:TestPoint_Loop_D1.80mm_Drill1.0mm_Beaded, F.Cu at (153.1, 76.7)
- added U1: ESP32-S3-WROOM-1-N16R2, MOD FILE:XCVR_ESP32-S3-WROOM-1-N16R2, F.Cu at (170.4, 67.0)
- added U2: SN65HVD72DR, Package_SO:SOIC-8_3.9x4.9mm_P1.27mm, F.Cu at (118.7, 113.0)
- added U3: LMR33620ADDA, Package_SO:Texas_HSOP-8-1EP_3.9x4.9mm_P1.27mm_ThermalVias, F.Cu at (108.1, 92.3)
- added U4: TPS7A2633DRVR, TPS7A2633DRVR:SON65P200X200X80-7N, F.Cu at (142.8, 81.2)
- added U5: CP2102N-QFN28, Package_DFN_QFN:QFN-28-1EP_5x5mm_P0.5mm_EP3.35x3.35mm, F.Cu at (142.2, 108.6)
- added kibuzzard-66F3845E: G***, kibuzzard-66F3845E, F.Cu at (81.5, 118.5)
- added kibuzzard-66F38482: G***, kibuzzard-66F38482, F.Cu at (85.9, 97.1)
- added kibuzzard-66F38482: G***, kibuzzard-66F38482, F.Cu at (179.1, 124.9)
- added kibuzzard-66F38482: G***, kibuzzard-66F38482, F.Cu at (104.0, 125.0)
- added kibuzzard-66F384BF: G***, kibuzzard-66F384BF, F.Cu at (78.6, 81.6)
- added kibuzzard-66F384E4: G***, kibuzzard-66F384E4, F.Cu at (121.7, 55.9)
- added kibuzzard-66F384FE: G***, kibuzzard-66F384FE, F.Cu at (96.7, 55.9)
- added kibuzzard-66F38519: G***, kibuzzard-66F38519, F.Cu at (109.6, 55.9)
- added kibuzzard-66F389F0: G***, kibuzzard-66F389F0, F.Cu at (138.9, 65.7)
Other:
- board outline added: 128 x 85 mm
- board text added: "Made in Cambodia"
- board text added: "Main HydroB"
