File: HydroB V2_Mainboard/LCD High Revolution.kicad_pcb (KiCad board)
At the start: 2 copper layers, 128 x 85 mm, 83 parts, among them J1 Conn_01x02_Pin, J10 USB_C_2.0, J2 Conn_01x02_Pin, J3 SENSOR, J4 Conn_01x02_Pin, J6 12V, J7 Conn_01x02_Pin, J8 LCD, J9 SENSOR, Q1 S8050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

Commit message: PCB placement and ERC
Parts:
- removed F1: Fuse, Fuse:Fuse_0805_2012Metric
- removed U5: CP2102N-QFN28, Package_DFN_QFN:QFN-28-1EP_5x5mm_P0.5mm_EP3.35x3.35mm
- removed kibuzzard-66F389F0: G***, kibuzzard-66F389F0
- added C19: 1uF, Capacitor_SMD:C_0603_1608Metric, F.Cu at (162.9, 106.9)
- added C20: 0.1uF, Capacitor_SMD:C_0603_1608Metric, F.Cu at (149.9, 105.1)
- added R17: 1k, Resistor_SMD:R_0603_1608Metric, F.Cu at (156.7, 116.4)
- added R2: 330, Resistor_SMD:R_0603_1608Metric, F.Cu at (149.9, 107.1)
- added SW3: SW_Push, Button_Switch_THT:SW_Tactile_SPST_Angled_PTS645Vx39-2LFS, F.Cu at (143.8, 136.1)
- added U6: SRV05-4, Package_TO_SOT_SMD:SOT-23-6, F.Cu at (145.3, 106.9)
- added U7: CP2104, Package_DFN_QFN:QFN-24-1EP_4x4mm_P0.5mm_EP2.6x2.6mm, F.Cu at (156.5, 109.7)
- added kibuzzard-66F769D4: G***, kibuzzard-66F769D4, F.Cu at (141.5, 130.0)
- added kibuzzard-67033E48: G***, kibuzzard-67033E48, F.Cu at (164.6, 70.4)
- added kibuzzard-67033E7E: G***, kibuzzard-67033E7E, F.Cu at (157.4, 128.6)
- C17: value 100nF -> 1uF
- C18: value 100nF -> 0.1uF
- L1: value 10uH -> 2.2uH
- R13: value 43.2k -> 24.9k
- moved J10 75.9 mm to (157.4, 133.9), turned to 0 degrees
- moved R18 36.3 mm to (156.6, 83.7)
- moved D8 27.2 mm to (129.4, 102.6), turned to -90 degrees
- moved R32 24.5 mm to (131.8, 102.6), turned to -90 degrees
- moved SW2 22.6 mm to (164.7, 73.8)
- moved C14 22.6 mm to (129.3, 96.0), turned to 90 degrees
- moved C1 21.8 mm to (135.0, 65.3)
- moved C2 21.8 mm to (134.2, 61.9)
- moved C3 21.8 mm to (136.2, 61.9)
- moved R30 21.8 mm to (135.0, 67.6)
- moved U1 21.8 mm to (148.7, 66.8)
- moved TP3 21.5 mm to (131.6, 71.7)
- moved TP4 21.5 mm to (131.6, 76.3)
- moved D1 21.3 mm to (165.1, 64.9)
- moved R1 21.3 mm to (162.8, 64.9)
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Connections:
- C14 pad 1: +5V -> VBUS
- C16 pad 2: +5V -> VBUS
- C17 pad 1: +5V -> GND
- C17 pad 2: GND -> /Mainboard/UART/VIO
- C18 pad 1: +3.3V -> GND
- C18 pad 2: GND -> /Mainboard/UART/VIO
- D3 pad 1: GND -> /Mainboard/UART/~{TXT}
- D5 pad 1: GND -> /Mainboard/UART/~{RXT}
- J10 pad A4: /Mainboard/UART/VBUS -> VBUS
- J10 pad A9: /Mainboard/UART/VBUS -> VBUS
- J10 pad B4: /Mainboard/UART/VBUS -> VBUS
- J10 pad B9: /Mainboard/UART/VBUS -> VBUS
- J10 pad S1: GND -> GNDPWR
- J7 pad 1: +3.3V -> VBUS
- R18 pad 2: /Mainboard/UART/~{RESET} -> Net-(U1-IO45)
- R21 pad 2: /Mainboard/UART/~{TXT} -> /Mainboard/UART/VIO
- R22 pad 2: /Mainboard/UART/~{RXT} -> /Mainboard/UART/VIO
- U1 pad 26: unconnected-(U1-IO45-Pad26) -> Net-(U1-IO45)
- U4 pad 4: +5V -> VBUS
- U4 pad 6: +5V -> VBUS
