File: HydroB V2_Mainboard/UART.kicad_sch (KiCad schematic)
At the start: 17 parts, among them J10 USB_C_2.0, Q3 1P, Q4 1P, U5 CP2102N-QFN28

Commit message: PCB placement and ERC
Parts:
- removed D6: LEDR, LED_SMD:LED_0603_1608Metric, symbol Device:LED_Small
- removed F1: Fuse, Fuse:Fuse_0805_2012Metric, symbol Device:Fuse
- removed J10: USB_C_2.0, Connector_USB:USB_C_Receptacle_Palconn_UTC16-G, symbol Connector:USB_C_Receptacle_USB2.0
- removed R18: 10k, Resistor_SMD:R_0603_1608Metric, symbol Device:R_Small
- removed R23: 1k, Resistor_SMD:R_0603_1608Metric, symbol Device:R_Small
- removed U5: CP2102N-QFN28, Package_DFN_QFN:QFN-28-1EP_5x5mm_P0.5mm_EP3.35x3.35mm, symbol Interface_USB:CP2102N-Axx-xQFN28
- added C19: 1uF, Capacitor_SMD:C_0603_1608Metric, symbol Device:C_Small
- added C20: 0.1uF, Capacitor_SMD:C_0603_1608Metric, symbol Device:C_Small
- added J5: USB_C_Receptacle_USB2.0_16P, symbol Connector:USB_C_Receptacle_USB2.0_16P
- added R17: 1k, Resistor_SMD:R_0603_1608Metric, symbol Device:R_Small
- added R2: 330, Resistor_SMD:R_0603_1608Metric, symbol Device:R_Small
- added U6: SRV05-4, Package_TO_SOT_SMD:SOT-23-6, symbol Power_Protection:SRV05-4
- added U7: CP2104, Package_DFN_QFN:QFN-24-1EP_4x4mm_P0.5mm_EP2.6x2.6mm, symbol Interface_USB:CP2104
- C17: value 100nF -> 1uF
- C18: value 100nF -> 0.1uF
Connections:
- net +3.3V is gone; now on net GND: C18.1
- net GND: now also C17.1, C19.1, C20.2, J5.A1 (GND), J5.A12 (GND), J5.B1 (GND), J5.B12 (GND), R2.1, U7.2 (GND), U7.25 (GND); no longer C17.2, C18.2, D3.1 (K), D5.1 (K)
- net UART_RX: now also U7.20 (RXD)
- net UART_TX: now also U7.21 (TXD)
- net USB_D+: now also J5.A6 (D+), J5.B6 (D+), U6.1 (IO1), U7.3 (D+)
- net USB_D-: now also J5.A7 (D-), J5.B7 (D-), U6.3 (IO2), U7.4 (D-)
- net VBUS: now also C16.2, J5.A4 (VBUS), J5.A9 (VBUS), J5.B4 (VBUS), J5.B9 (VBUS), U6.5 (VP), U7.7 (REGIN), U7.8 (VBUS)
- net ~{DTR}: now also U7.23 (~{DTR})
- net ~{RST}: now also U7.19 (~{RTS})
- net ~{RXT}: now also D5.1 (K), U7.13 (RXT/GPIO.1); no longer R22.2
- net ~{TXT}: now also D3.1 (K), U7.14 (TXT/GPIO.0); no longer R21.2
- removed net +5V: C16.2, C17.1
- new net: R17.1, U7.9 (~{RST})
- new net: C19.2, U7.16 (VPP)
- new net GNDPWR: C20.1, J5.S1 (SHIELD), R2.2, U6.2 (VN)
- new net VIO: C17.2, C18.2, R17.2, R21.2, R22.2, U7.5 (VIO), U7.6 (VDD)
- no-connect marks 18 -> 14
Other:
- note added: "shield to signal GND connection"
- company: (none) -> UART
- title: (none) -> Prak Chilifong
- moved on the sheet: D3, D5, Q3, Q4, R19, R20, R21, R22
