File: HydroB V2_Mainboard/LCD High Revolution.kicad_sch (KiCad schematic)
At the start: 0 parts

Commit message: Mainboard schematic update
Other:
- sheet LCD renamed Mainboard
- sheet Mainboard: file LCD.kicad_sch -> Mainboard.kicad_sch
- note added: "Sheet 1: Root Sheet 2: Project review of ESP32-S3 Sheet 3: Modbus Sheet 4: Power Supply Sheet 5: LED Indicator"
- note removed: "Sheet 1: Root Sheet 2: Project review of LCD Sheet 3: ESP32-S3 Sheet 4: LCD Connector Sheet 5: Boost LED converter Sheet 6: Step_LED Power Sheet 7: USB type and the reset and boot button Sheet 8: Power Supply"
Changed lines of the file:
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@@
 	(generator_version "8.0")
 	(paper "A4")
-	(text "Sheet 1: Root\n\nSheet 2: Project review of LCD\n\nSheet 3: ESP32-S3\n\nSheet 4: LCD Connector\n\nSheet 5: Boost LED converter\n\nSheet 6: Step_LED Power\n\nSheet 7: USB type and the reset and boot button\n\nSheet 8: Power Supply\n"
+	(text "Sheet 1: Root\n\nSheet 2: Project review of ESP32-S3\n\nSheet 3: Modbus\n\nSheet 4: Power Supply\n\nSheet 5: LED Indicator\n"
 		(exclude_from_sim no)
-		(at 18.542 64.262 0)
+		(at 24.892 71.882 0)
 		(effects
 			(font
@@
 	)
 	(sheet
-		(at 19.05 22.86)
+		(at 25.4 30.48)
 		(size 43.18 30.48)
 		(fields_autoplaced yes)
@@
 			(color 255 255 194 1.0000)
 		)
-		(property "Sheetname" "LCD"
-			(at 19.05 22.1484 0)
+		(property "Sheetname" "Mainboard"
+			(at 25.4 29.7684 0)
 			(effects
 				(font
@@
 			)
 		)
-		(property "Sheetfile" "LCD.kicad_sch"
-			(at 19.05 53.9246 0)
+		(property "Sheetfile" "Mainboard.kicad_sch"
+			(at 25.4 61.5446 0)
 			(effects
 				(font

Commit message: PCB placement and ERC
Other:
- note added: "Sheet 1: Root Sheet 2: Mainboard Sheet 3: Modbus Sheet 4: Power Supply Sheet 5: LED Indicator Sheet 6: UART"
- note removed: "Sheet 1: Root Sheet 2: Project review of ESP32-S3 Sheet 3: Modbus Sheet 4: Power Supply Sheet 5: LED Indicator"
- company: (none) -> Root
- title: (none) -> Prak Chilifong
Changed lines of the file:
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@@
 	(generator_version "8.0")
 	(paper "A4")
-	(text "Sheet 1: Root\n\nSheet 2: Project review of ESP32-S3\n\nSheet 3: Modbus\n\nSheet 4: Power Supply\n\nSheet 5: LED Indicator\n"
+	(title_block
+		(title "Prak Chilifong")
+		(date "2024-10-06")
+		(rev "2.0")
+		(company "Root")
+		(comment 1 "Mainboard PCB")
+	)
+	(text "Sheet 1: Root\n\nSheet 2: Mainboard\n\nSheet 3: Modbus\n\nSheet 4: Power Supply\n\nSheet 5: LED Indicator\n\nSheet 6: UART\n"
 		(exclude_from_sim no)
 		(at 24.892 71.882 0)

Commit message: PCB placement and RUN ERC
Other:
- note added: "${ISSUE_DATE} V1-Rev${REVISION}"
- note added: "${TITLE}"
- note added: "........................................................"
- note added: "1"
- note added: "10"
- note added: "11"
- note added: "12"
- note added: "13"
- note added: "14"
- note added: "15"
- note added: "16"
- note added: "17"
- note added: "18"
- note added: "19"
- note added: "2"
- note added: "20"
- note added: "3"
- note added: "4"
- note added: "5"
- note added: "6"
- note added: "7"
- note added: "8"
- note added: "9"
- note added: "BLOCK DIAGRAM"
- note added: "COVER PAGE"
- note added: "Chiptree Lab"
- note added: "Index"
- note added: "LED"
- note added: "MCU"
- note added: "Modbus"
- note added: "Page"
- note added: "Power Supply"
- note added: "RELEASED YYYY-MM-DD"
- note added: "Rendered image 1"
- note added: "Rendered image 2"
- note added: "UART"
- note removed: "Sheet 1: Root Sheet 2: Mainboard Sheet 3: Modbus Sheet 4: Power Supply Sheet 5: LED Indicator Sheet 6: UART"
